File: hunity-gru-master/hunity-gru-master.kicad_pcb (KiCad board)
At the start: 2 copper layers, 56 x 21 mm, 12 parts, among them J1 Conn_01x10_Pin, J2 Conn_01x10_Socket, U1 BME280, U2 AP2112K-3.3

Commit message: labelling+generating production files
Other:
- board text added: "5V"
- board text added: "EN1"
- board text added: "EN2"
- board text added: "EN3"
- board text added: "EN4"
- board text added: "EN5"
- board text added: "EN6"
- board text added: "GND"
- board text added: "SCL"
- board text added: "SDA"
